File: c64-wedge-psu-pcb.kicad_pcb (KiCad board)
At the start: 2 copper layers, 70 x 54 mm, 22 parts, among them U1 LM2576T-ADJ

Commit message: Updates
Parts:
- moved D3 12.7 mm to (100.3, 76.2), turned to -90 degrees
- moved D4 12.7 mm to (95.2, 76.2), turned to -90 degrees
- moved R2 12.0 mm to (117.3, 97.8), turned to -90 degrees
- moved R1 10.5 mm to (114.3, 105.4), turned to 90 degrees
- moved C6 7.84 mm to (157.5, 106.7), turned to 90 degrees
- moved U1 6.80 mm to (108.8, 99.1), turned to 180 degrees
- moved C3 2.69 mm to (153.0, 97.2), turned to 90 degrees
- moved L2 1.41 mm to (150.5, 105.4)
Connections:
- D3 pad 1: /GND -> Net-(D1-A)
- D3 pad 2: Net-(D1-A) -> /GND
- D4 pad 1: /GND -> Net-(D2-A)
- D4 pad 2: Net-(D2-A) -> /GND
Routing:
- net Net-(D1-K): track 94.4 -> 49.8 mm
- net Net-(C2-Pad1): track 42.8 -> 57.6 mm
- net /+5VDC: track 58.6 -> 55.4 mm
- net Net-(D5-K): track 55.0 -> 52.6 mm
- net Net-(D2-A): track 27.1 -> 28.9 mm
- net Net-(U1-FB): track 14.6 -> 15.5 mm
Other:
- board text added: "(GRN)"
- board text added: "(WHT)"
- board text added: "V2.0 - 03/2026"
- board text removed: "V1.4- 03/2026"

Commit message: updates
Parts:
- L2: value 20uH -> 22uH
- moved C4 19.0 mm to (120.0, 87.6), turned to -90 degrees
- moved C6 7.00 mm to (157.0, 99.7), turned to -90 degrees
- moved C5 3.72 mm to (137.8, 89.5), turned to 180 degrees
Routing:
- net Net-(D1-K): track 49.8 -> 45.3 mm
- net Net-(C2-Pad1): track 57.6 -> 60.8 mm
