File: c64-wedge-psu-pcb.kicad_sch (KiCad schematic)
At the start: 16 parts, among them U1 LM2576T-5

Commit message: Update to 1.4
Parts:
- removed D1: 6A, Diode_THT:Diode_Bridge_Vishay_KBPC6, symbol Diode_Bridge:VS-KBPC801
- added C4, C5, C6: 0.1uF, Capacitor_THT:C_Disc_D3.0mm_W1.6mm_P2.50mm, symbol c64-wedge-psu-pcb-rescue:CP-Device
- added D1, D2, D3, D4: SB540, Diode_THT:D_DO-201AD_P12.70mm_Horizontal, symbol Device:D_Schottky
- D5: renamed from D2; value 5A -> SB540
- H1, H2, H3, H4: footprint Connector_Wire:SolderWirePad_1x01_Drill2mm -> Connector_Wire:SolderWire-1.5sqmm_1x01_D1.7mm_OD3.9mm
- L1: value 150uH -> 100uH
- L2: value 22uH -> 20uH
- R1: renamed from R3; value 10K -> 1k
- R2: renamed from R1; value 150 -> 3.2k
- U1: value LM2576T-5 -> LM2576T-ADJ; footprint Package_TO_SOT_THT:TO-220-5_P3.4x3.8mm_StaggerEven_Lead7.13mm_TabDown -> Package_TO_SOT_THT:TO-220-5_P3.4x3.7mm_StaggerEven_Lead3.8mm_Vertical
- renumbered R2 to R3
Connections:
- net +5VDC: now also C6.1
- net GND: now also C4.2, C5.2, C6.2, D3.2 (A), D4.2 (A)
- net at C1.1, U1.1 (VIN): now also C4.1, D1.1 (K), D2.1 (K)
- net at C2.1, L1.2, L2.1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: now also C5.1
- net at H1.1: now also D2.2 (A), D4.1 (K)
- net at H2.1: now also D1.2 (A), D3.1 (K)
Other:
- moved on the sheet: C1, C2, C3, H1, H2, H3, H4, L1, LED1, R1, R2, R3

Commit message: fixed
Parts:
- C1, C2, C3: symbol c64-wedge-psu-pcb-rescue:CP-Device -> Device:C_Polarized
- C4, C5, C6: symbol c64-wedge-psu-pcb-rescue:CP-Device -> Device:C
- U1: symbol Regulator_Switching:LM2576T-5 -> Regulator_Switching:LM2576T-ADJ
Changed lines of the file:
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@@
 	)
 	(symbol
-		(lib_id "Regulator_Switching:LM2576T-5")
+		(lib_id "Regulator_Switching:LM2576T-ADJ")
 		(at 116.84 95.25 0)
 		(unit 1)
@@
 		)
 		(property "Value" "LM2576T-ADJ"
-			(at 116.84 88.2396 0)
-			(effects
-				(font
-					(size 1.27 1.27)
-				)
+			(at 116.84 88.9 0)
+			(effects
+				(font
+					(size 1.27 1.27)
+				)
+				(justify left)
 			)
 		)
@@
 			)
 		)
-		(property "Description" ""
+		(property "Description" "Adjustable Output Voltage, 3A SIMPLE SWITCHER® Step-Down Voltage Regulator, TO-220-5"
 			(at 116.84 95.25 0)
 			(effects
@@
 	)
 	(symbol
-		(lib_id "c64-wedge-psu-pcb-rescue:CP-Device")
+		(lib_id "Device:C_Polarized")
 		(at 153.67 102.87 0)
 		(unit 1)
@@
 			)
 		)
-		(property "Description" ""
+		(property "Description" "Polarized capacitor"
 			(at 153.67 102.87 0)
 			(effects
@@
 	)
 	(symbol
-		(lib_id "c64-wedge-psu-pcb-rescue:CP-Device")
+		(lib_id "Device:C_Polarized")
 		(at 92.71 100.33 0)
 		(unit 1)
@@
 			)
 		)
-		(property "Description" ""
+		(property "Description" "Polarized capacitor"
 			(at 92.71 100.33 0)
 			(effects
@@
 	)
 	(symbol
-		(lib_id "c64-wedge-psu-pcb-rescue:CP-Device")
+		(lib_id "Device:C_Polarized")
 		(at 199.39 100.33 0)
 		(unit 1)
@@
 			)
 		)
-		(property "Description" ""
+		(property "Description" "Polarized capacitor"
 			(at 199.39 100.33 0)
 			(effects
@@
 	)
 	(symbol
-		(lib_id "c64-wedge-psu-pcb-rescue:CP-Device")
+		(lib_id "Device:C")
 		(at 78.74 100.33 0)
 		(unit 1)
@@
 		(fields_autoplaced yes)
 		(property "Reference" "C4"
-			(at 82.37 98.1709 0)
+			(at 82.55 99.0599 0)
 			(effects
 				(font
@@
 		)
 		(property "Value" "0.1uF"
-			(at 82.37 100.7109 0)
+			(at 82.55 101.5999 0)
 			(effects
 				(font
@@
 		)
 		(property "Footprint" "Capacitor_THT:C_Disc_D3.0mm_W1.6mm_P2.50mm"
-			(at 79.68 104.14 0)
+			(at 79.7052 104.14 0)
 			(effects
 				(font
@@
 			)
 		)
-		(property "Description" "HF decoupling; parallel to C1"
+		(property "Description" "Unpolarized capacitor"
 			(at 78.74 100.33 0)
 			(effects
@@
 	)
 	(symbol
-		(lib_id "c64-wedge-psu-pcb-rescue:CP-Device")
+		(lib_id "Device:C")
 		(at 142.24 102.87 0)
 		(unit 1)
@@
 		(fields_autoplaced yes)
 		(property "Reference" "C5"
-			(at 145.29 100.7109 0)
+			(at 146.05 101.5999 0)
 			(effects
 				(font
@@
 		)
 		(property "Value" "0.1uF"
-			(at 145.29 103.2509 0)
+			(at 146.05 104.1399 0)
 			(effects
 				(font
@@
 		)
 		(property "Footprint" "Capacitor_THT:C_Disc_D3.0mm_W1.6mm_P2.50mm"
-			(at 143.18 106.68 0)
+			(at 143.2052 106.68 0)
 			(effects
 				(font
@@
 			)
 		)
-		(property "Description" "HF decoupling; parallel to C2"
+		(property "Description" "Unpolarized capacitor"
 			(at 142.24 102.87 0)
 			(effects
@@
 	)
 	(symbol
-		(lib_id "c64-wedge-psu-pcb-rescue:CP-Device")
+		(lib_id "Device:C")
 		(at 186.69 100.33 0)
 		(unit 1)
@@
 		(fields_autoplaced yes)
 		(property "Reference" "C6"
-			(at 190.5 98.1709 0)
+			(at 190.5 99.0599 0)
 			(effects
 				(font
@@
 		)
 		(property "Value" "0.1uF"
-			(at 190.5 100.7109 0)
+			(at 190.5 101.5999 0)
 			(effects
 				(font
@@
 		)
 		(property "Footprint" "Capacitor_THT:C_Disc_D3.0mm_W1.6mm_P2.50mm"
-			(at 187.63 104.14 0)
+			(at 187.6552 104.14 0)
 			(effects
 				(font
@@
 			)
 		)
-		(property "Description" "HF decoupling; parallel to C3"
+		(property "Description" "Unpolarized capacitor"
 			(at 186.69 100.33 0)
 			(effects

Commit message: updates
Parts:
- L2: value 20uH -> 22uH
Changed lines of the file:
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@@
 			)
 		)
-		(property "Description" "Adjustable Output Voltage, 3A SIMPLE SWITCHER® Step-Down Voltage Regulator, TO-220-5"
+		(property "Description" "LM2576T-ADJ"
 			(at 116.84 95.25 0)
 			(effects
@@
 			)
 		)
-		(property "Datasheet" "~"
+		(property "Datasheet" "https://yageogroup.com/content/datasheet/asset/file/DATASHEET_P596"
 			(at 133.35 97.79 0)
 			(effects
@@
 			)
 		)
-		(property "Description" ""
+		(property "Description" "Pulse PE-92108KNL (100µH, KM-4)"
 			(at 133.35 97.79 0)
 			(effects
@@
 			)
 		)
-		(property "Description" ""
+		(property "Description" "SB540-E3/54"
 			(at 129.54 104.14 0)
 			(effects
@@
 			)
 		)
-		(property "Description" "Polarized capacitor"
+		(property "Description" "UPW1E222MHD"
 			(at 153.67 102.87 0)
 			(effects
@@
 			)
 		)
-		(property "Description" "Bridge: band to +"
+		(property "Description" "SB540-E3/54"
 			(at 68.58 88.9 0)
 			(effects
@@
 			)
 		)
-		(property "Description" "Bridge: band to +"
+		(property "Description" "SB540-E3/54"
 			(at 68.58 96.52 0)
 			(effects
@@
 			)
 		)
-		(property "Description" "Bridge: band to -"
+		(property "Description" "SB540-E3/54"
 			(at 60.96 88.9 0)
 			(effects
@@
 			)
 		)
-		(property "Description" "Bridge: band to -"
+		(property "Description" "SB540-E3/54"
 			(at 60.96 96.52 0)
 			(effects
@@
 			)
 		)
-		(property "Description" "Polarized capacitor"
+		(property "Description" "UHE1E472MHD"
 			(at 92.71 100.33 0)
 			(effects
@@
 			)
 		)
-		(property "Description" "Polarized capacitor"
+		(property "Description" "UHE1E221MPD"
 			(at 199.39 100.33 0)
 			(effects
@@
 			)
 		)
-		(property "Value" "20uH"
+		(property "Value" "22uH"
 			(at 177.8 90.1954 90)
 			(effects
@@
 			)
 		)
-		(property "Datasheet" "~"
+		(property "Datasheet" "https://www.bourns.com/docs/product-datasheets/6100.pdf"
 			(at 177.8 92.71 0)
 			(effects
@@
 			)
 		)
-		(property "Description" ""
+		(property "Description" "Bourns 6100-220K-RC (22µH, 4.52A)"
 			(at 177.8 92.71 0)
 			(effects
